File: hardware/main-board/main-board.kicad_pcb (KiCad board)
At the start: 4 copper layers, 105 x 38 mm, 101 parts, among them J1 USB_C_Receptacle_USB2.0, J2 DNI, J3 Display Connector, J4 Conn_01x04, SW1 SW_Push, SW2 SW_Push, SW3 SW_Push, SW4 SW_Push, SW5 SW_Detect, SW6 SW_Boot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

Commit message: Final routing and silkscreen tweaks
Fixed some trace sizing cruft
Swapped TVS diode footprints for better pin 1 clarity
Routing:
- added copper zone on B.Cu, net +5V
